Commit message: Adds mesh for vacuum gripper

File: robotiq_vacuum_gripper_description/urdf/epick.urdf.xacro (robot description, xacro)
@@ -12,5 +12,5 @@
             <mesh filename="package://robotiq_vacuum_gripper_description/urdf/meshes/epick.stl" scale="0.001 0.001 0.001"/>
         </geometry>
-      <material name="black"/>
+      <material name="metal_grey"/>
     </visual>
     <collision>
